Commit message: Update to add TRACK link and joints

File: rtr_double_arm_v7_description/urdf/BASE-AGX.urdf.xacro (robot description, xacro)
@@ -12,116 +12,4 @@
   </material>
   <!-- Link -->
-  <link name="WHEEL_L0">
-    <visual>
-      <origin rpy="${-M_PI/2} 0 0"/>
-      <material name="wheel_color"/>
-      <geometry>
-        <cylinder radius="0.2" length="0.25"/>
-      </geometry>
-    </visual>
-    <inertial>
-      <mass value="13.25" />
-      <origin xyz="0.0 0.0 0.0" rpy="0 -0 0" />
-      <inertia ixx="0.2015" ixy="0.0" ixz="0.0" iyy="0.265" iyz="0.0" izz="0.2015" />
-    </inertial>
-  </link>
-  <link name="WHEEL_L1">
-    <visual>
-      <origin rpy="${-M_PI/2} 0 0"/>
-      <material name="wheel_color"/>
-      <geometry>
-        <cylinder radius="0.2" length="0.25"/>
-      </geometry>
-    </visual>
-    <inertial>
-      <mass value="13.25" />
-      <origin xyz="0.0 0.0 0.0" rpy="0 -0 0" />
-      <inertia ixx="0.2015" ixy="0.0" ixz="0.0" iyy="0.265" iyz="0.0" izz="0.2015" />
-    </inertial>
-  </link>
-  <link name="WHEEL_L2">
-    <visual>
-      <origin rpy="${-M_PI/2} 0 0"/>
-      <material name="wheel_color"/>
-      <geometry>
-        <cylinder radius="0.2" length="0.25"/>
-      </geometry>
-    </visual>
-    <inertial>
-      <mass value="13.25" />
-      <origin xyz="0.0 0.0 0.0" rpy="0 -0 0" />
-      <inertia ixx="0.2015" ixy="0.0" ixz="0.0" iyy="0.265" iyz="0.0" izz="0.2015" />
-    </inertial>
-  </link>
-  <link name="WHEEL_L3">
-    <visual>
-      <origin rpy="${-M_PI/2} 0 0"/>
-      <material name="wheel_color"/>
-      <geometry>
-        <cylinder radius="0.2" length="0.25"/>
-      </geometry>
-    </visual>
-    <inertial>
-      <mass value="13.25" />
-      <origin xyz="0.0 0.0 0.0" rpy="0 -0 0" />
-      <inertia ixx="0.2015" ixy="0.0" ixz="0.0" iyy="0.265" iyz="0.0" izz="0.2015" />
-    </inertial>
-  </link>
-  <link name="WHEEL_R0">
-    <visual>
-      <origin rpy="${-M_PI/2} 0 0"/>
-      <material name="wheel_color"/>
-      <geometry>
-        <cylinder radius="0.2" length="0.25"/>
-      </geometry>
-    </visual>
-    <inertial>
-      <mass value="13.25" />
-      <origin xyz="0.0 0.0 0.0" rpy="0 -0 0" />
-      <inertia ixx="0.2015" ixy="0.0" ixz="0.0" iyy="0.265" iyz="0.0" izz="0.2015" />
-    </inertial>
-  </link>
-  <link name="WHEEL_R1">
-    <visual>
-      <origin rpy="${-M_PI/2} 0 0"/>
-      <material name="wheel_color"/>
-      <geometry>
-        <cylinder radius="0.2" length="0.25"/>
-      </geometry>
-    </visual>
-    <inertial>
-      <mass value="13.25" />
-      <origin xyz="0.0 0.0 0.0" rpy="0 -0 0" />
-      <inertia ixx="0.2015" ixy="0.0" ixz="0.0" iyy="0.265" iyz="0.0" izz="0.2015" />
-    </inertial>
-  </link>
-  <link name="WHEEL_R2">
-    <visual>
-      <origin rpy="${-M_PI/2} 0 0"/>
-      <material name="wheel_color"/>
-      <geometry>
-        <cylinder radius="0.2" length="0.25"/>
-      </geometry>
-    </visual>
-    <inertial>
-      <mass value="13.25" />
-      <origin xyz="0.0 0.0 0.0" rpy="0 -0 0" />
-      <inertia ixx="0.2015" ixy="0.0" ixz="0.0" iyy="0.265" iyz="0.0" izz="0.2015" />
-    </inertial>
-  </link>
-  <link name="WHEEL_R3">
-    <visual>
-      <origin rpy="${-M_PI/2} 0 0"/>
-      <material name="wheel_color"/>
-      <geometry>
-        <cylinder radius="0.2" length="0.25"/>
-      </geometry>
-    </visual>
-    <inertial>
-      <mass value="13.25" />
-      <origin xyz="0.0 0.0 0.0" rpy="0 -0 0" />
-      <inertia ixx="0.2015" ixy="0.0" ixz="0.0" iyy="0.265" iyz="0.0" izz="0.2015" />
-    </inertial>
-  </link>
   <link name="WIRE_GUARD_L">
     <visual>
@@ -184,55 +72,4 @@
     </inertial>
   </link>
-  <!-- Joint -->
-  <joint name="WHEEL_L0" type="continuous">
-    <origin xyz="0.74 0.6 -0.295" rpy="0.0 -0.0 0.0" />
-    <parent link="TFRAME" />
-    <child link="WHEEL_L0" />
-    <axis xyz="0 1 0"/>
-  </joint>
-  <xacro:joint_velocity_trans_v0 name="WHEEL_L0"/>
-  <joint name="WHEEL_L1" type="continuous">
-    <origin xyz="0.26 0.6 -0.295" rpy="0.0 -0.0 0.0" />
-    <parent link="TFRAME" />
-    <child link="WHEEL_L1" />
-    <axis xyz="0 1 0"/>
-  </joint>
-  <joint name="WHEEL_L2" type="continuous">
-    <origin xyz="-0.22 0.6 -0.295" rpy="0.0 -0.0 0.0" />
-    <parent link="TFRAME" />
-    <child link="WHEEL_L2" />
-    <axis xyz="0 1 0"/>
-  </joint>
-  <joint name="WHEEL_L3" type="continuous">
-    <origin xyz="-0.7 0.6 -0.295" rpy="0.0 -0.0 0.0" />
-    <parent link="TFRAME" />
-    <child link="WHEEL_L3" />
-    <axis xyz="0 1 0"/>
-  </joint>
-  <joint name="WHEEL_R0" type="continuous">
-    <origin xyz="0.74 -0.6 -0.295" rpy="0.0 -0.0 0.0" />
-    <parent link="TFRAME" />
-    <child link="WHEEL_R0" />
-    <axis xyz="0 -1 0"/>
-  </joint>
-  <xacro:joint_velocity_trans_v0 name="WHEEL_R0"/>
-  <joint name="WHEEL_R1" type="continuous">
-    <origin xyz="0.26 -0.6 -0.295" rpy="0.0 -0.0 0.0" />
-    <parent link="TFRAME" />
-    <child link="WHEEL_R1" />
-    <axis xyz="0 1 0"/>
-  </joint>
-  <joint name="WHEEL_R2" type="continuous">
-    <origin xyz="-0.22 -0.6 -0.295" rpy="0.0 -0.0 0.0" />
-    <parent link="TFRAME" />
-    <child link="WHEEL_R2" />
-    <axis xyz="0 1 0"/>
-  </joint>
-  <joint name="WHEEL_R3" type="continuous">
-    <origin xyz="-0.7 -0.6 -0.295" rpy="0.0 -0.0 0.0" />
-    <parent link="TFRAME" />
-    <child link="WHEEL_R3" />
-    <axis xyz="0 1 0"/>
-  </joint>
   <joint name="WIRE_GUARD_L" type="fixed">
     <origin xyz="0.02 0.61 -0.32" rpy="0.0 -0.0 0.0" />
@@ -245,3 +82,20 @@
     <child link="WIRE_GUARD_R" />
   </joint>
+  <link name="TRACK_L"/>
+  <joint name="TRACK_L" type="continuous">
+    <axis xyz="0 1 0"/>
+    <origin xyz="0.02 0.61 -0.32" rpy="0.0 -0.0 0.0" />
+    <parent link="TFRAME" />
+    <child link="TRACK_L" />
+  </joint>
+  <link name="TRACK_R"/>
+  <joint name="TRACK_R" type="continuous">
+    <axis xyz="0 -1 0"/>
+    <origin xyz="0.02 -0.61 -0.32" rpy="0.0 -0.0 0.0" />
+    <parent link="TFRAME" />
+    <child link="TRACK_R" />
+  </joint>
+  <!-- Transmission -->
+  <xacro:joint_velocity_trans_v0 name="TRACK_L"/>
+  <xacro:joint_velocity_trans_v0 name="TRACK_R"/>
 </robot>

Commit message: Fix AGX and AIST base urdf for joint names

File: rtr_double_arm_v7_description/urdf/BASE-AGX.urdf.xacro (robot description, xacro)
@@ -12,4 +12,116 @@
   </material>
   <!-- Link -->
+  <link name="WHEEL_L0">
+    <visual>
+      <origin rpy="${-M_PI/2} 0 0"/>
+      <material name="wheel_color"/>
+      <geometry>
+        <cylinder radius="0.2" length="0.25"/>
+      </geometry>
+    </visual>
+    <inertial>
+      <mass value="13.25" />
+      <origin xyz="0.0 0.0 0.0" rpy="0 -0 0" />
+      <inertia ixx="0.2015" ixy="0.0" ixz="0.0" iyy="0.265" iyz="0.0" izz="0.2015" />
+    </inertial>
+  </link>
+  <link name="WHEEL_L1">
+    <visual>
+      <origin rpy="${-M_PI/2} 0 0"/>
+      <material name="wheel_color"/>
+      <geometry>
+        <cylinder radius="0.2" length="0.25"/>
+      </geometry>
+    </visual>
+    <inertial>
+      <mass value="13.25" />
+      <origin xyz="0.0 0.0 0.0" rpy="0 -0 0" />
+      <inertia ixx="0.2015" ixy="0.0" ixz="0.0" iyy="0.265" iyz="0.0" izz="0.2015" />
+    </inertial>
+  </link>
+  <link name="WHEEL_L2">
+    <visual>
+      <origin rpy="${-M_PI/2} 0 0"/>
+      <material name="wheel_color"/>
+      <geometry>
+        <cylinder radius="0.2" length="0.25"/>
+      </geometry>
+    </visual>
+    <inertial>
+      <mass value="13.25" />
+      <origin xyz="0.0 0.0 0.0" rpy="0 -0 0" />
+      <inertia ixx="0.2015" ixy="0.0" ixz="0.0" iyy="0.265" iyz="0.0" izz="0.2015" />
+    </inertial>
+  </link>
+  <link name="WHEEL_L3">
+    <visual>
+      <origin rpy="${-M_PI/2} 0 0"/>
+      <material name="wheel_color"/>
+      <geometry>
+        <cylinder radius="0.2" length="0.25"/>
+      </geometry>
+    </visual>
+    <inertial>
+      <mass value="13.25" />
+      <origin xyz="0.0 0.0 0.0" rpy="0 -0 0" />
+      <inertia ixx="0.2015" ixy="0.0" ixz="0.0" iyy="0.265" iyz="0.0" izz="0.2015" />
+    </inertial>
+  </link>
+  <link name="WHEEL_R0">
+    <visual>
+      <origin rpy="${-M_PI/2} 0 0"/>
+      <material name="wheel_color"/>
+      <geometry>
+        <cylinder radius="0.2" length="0.25"/>
+      </geometry>
+    </visual>
+    <inertial>
+      <mass value="13.25" />
+      <origin xyz="0.0 0.0 0.0" rpy="0 -0 0" />
+      <inertia ixx="0.2015" ixy="0.0" ixz="0.0" iyy="0.265" iyz="0.0" izz="0.2015" />
+    </inertial>
+  </link>
+  <link name="WHEEL_R1">
+    <visual>
+      <origin rpy="${-M_PI/2} 0 0"/>
+      <material name="wheel_color"/>
+      <geometry>
+        <cylinder radius="0.2" length="0.25"/>
+      </geometry>
+    </visual>
+    <inertial>
+      <mass value="13.25" />
+      <origin xyz="0.0 0.0 0.0" rpy="0 -0 0" />
+      <inertia ixx="0.2015" ixy="0.0" ixz="0.0" iyy="0.265" iyz="0.0" izz="0.2015" />
+    </inertial>
+  </link>
+  <link name="WHEEL_R2">
+    <visual>
+      <origin rpy="${-M_PI/2} 0 0"/>
+      <material name="wheel_color"/>
+      <geometry>
+        <cylinder radius="0.2" length="0.25"/>
+      </geometry>
+    </visual>
+    <inertial>
+      <mass value="13.25" />
+      <origin xyz="0.0 0.0 0.0" rpy="0 -0 0" />
+      <inertia ixx="0.2015" ixy="0.0" ixz="0.0" iyy="0.265" iyz="0.0" izz="0.2015" />
+    </inertial>
+  </link>
+  <link name="WHEEL_R3">
+    <visual>
+      <origin rpy="${-M_PI/2} 0 0"/>
+      <material name="wheel_color"/>
+      <geometry>
+        <cylinder radius="0.2" length="0.25"/>
+      </geometry>
+    </visual>
+    <inertial>
+      <mass value="13.25" />
+      <origin xyz="0.0 0.0 0.0" rpy="0 -0 0" />
+      <inertia ixx="0.2015" ixy="0.0" ixz="0.0" iyy="0.265" iyz="0.0" izz="0.2015" />
+    </inertial>
+  </link>
   <link name="WIRE_GUARD_L">
     <visual>
@@ -72,4 +184,55 @@
     </inertial>
   </link>
+  <!-- Joint -->
+  <joint name="WHEEL_L0" type="continuous">
+    <origin xyz="0.74 0.6 -0.295" rpy="0.0 -0.0 0.0" />
+    <parent link="TFRAME" />
+    <child link="WHEEL_L0" />
+    <axis xyz="0 1 0"/>
+  </joint>
+  <xacro:joint_velocity_trans_v0 name="WHEEL_L0"/>
+  <joint name="WHEEL_L1" type="continuous">
+    <origin xyz="0.26 0.6 -0.295" rpy="0.0 -0.0 0.0" />
+    <parent link="TFRAME" />
+    <child link="WHEEL_L1" />
+    <axis xyz="0 1 0"/>
+  </joint>
+  <joint name="WHEEL_L2" type="continuous">
+    <origin xyz="-0.22 0.6 -0.295" rpy="0.0 -0.0 0.0" />
+    <parent link="TFRAME" />
+    <child link="WHEEL_L2" />
+    <axis xyz="0 1 0"/>
+  </joint>
+  <joint name="WHEEL_L3" type="continuous">
+    <origin xyz="-0.7 0.6 -0.295" rpy="0.0 -0.0 0.0" />
+    <parent link="TFRAME" />
+    <child link="WHEEL_L3" />
+    <axis xyz="0 1 0"/>
+  </joint>
+  <joint name="WHEEL_R0" type="continuous">
+    <origin xyz="0.74 -0.6 -0.295" rpy="0.0 -0.0 0.0" />
+    <parent link="TFRAME" />
+    <child link="WHEEL_R0" />
+    <axis xyz="0 -1 0"/>
+  </joint>
+  <xacro:joint_velocity_trans_v0 name="WHEEL_R0"/>
+  <joint name="WHEEL_R1" type="continuous">
+    <origin xyz="0.26 -0.6 -0.295" rpy="0.0 -0.0 0.0" />
+    <parent link="TFRAME" />
+    <child link="WHEEL_R1" />
+    <axis xyz="0 1 0"/>
+  </joint>
+  <joint name="WHEEL_R2" type="continuous">
+    <origin xyz="-0.22 -0.6 -0.295" rpy="0.0 -0.0 0.0" />
+    <parent link="TFRAME" />
+    <child link="WHEEL_R2" />
+    <axis xyz="0 1 0"/>
+  </joint>
+  <joint name="WHEEL_R3" type="continuous">
+    <origin xyz="-0.7 -0.6 -0.295" rpy="0.0 -0.0 0.0" />
+    <parent link="TFRAME" />
+    <child link="WHEEL_R3" />
+    <axis xyz="0 1 0"/>
+  </joint>
   <joint name="WIRE_GUARD_L" type="fixed">
     <origin xyz="0.02 0.61 -0.32" rpy="0.0 -0.0 0.0" />
@@ -82,20 +245,3 @@
     <child link="WIRE_GUARD_R" />
   </joint>
-  <link name="TRACK_L"/>
-  <joint name="TRACK_L" type="continuous">
-    <axis xyz="0 1 0"/>
-    <origin xyz="0.02 0.61 -0.32" rpy="0.0 -0.0 0.0" />
-    <parent link="TFRAME" />
-    <child link="TRACK_L" />
-  </joint>
-  <link name="TRACK_R"/>
-  <joint name="TRACK_R" type="continuous">
-    <axis xyz="0 -1 0"/>
-    <origin xyz="0.02 -0.61 -0.32" rpy="0.0 -0.0 0.0" />
-    <parent link="TFRAME" />
-    <child link="TRACK_R" />
-  </joint>
-  <!-- Transmission -->
-  <xacro:joint_velocity_trans_v0 name="TRACK_L"/>
-  <xacro:joint_velocity_trans_v0 name="TRACK_R"/>
 </robot>

File: rtr_double_arm_v7_description/urdf/BASE-AIST.urdf.xacro (robot description, xacro)
@@ -72,7 +72,4 @@
     </inertial>
   </link>
-  <!-- Transmission -->
-  <xacro:joint_velocity_trans_v0 name="TRACK_L"/>
-  <xacro:joint_velocity_trans_v0 name="TRACK_R"/>
   <joint name="WIRE_GUARD_L" type="fixed">
     <origin xyz="0.02 0.61 -0.32" rpy="0.0 -0.0 0.0" />
@@ -85,3 +82,20 @@
     <child link="WIRE_GUARD_R" />
   </joint>
+  <link name="TRACK_L"/>
+  <joint name="TRACK_L" type="continuous">
+    <axis xyz="0 1 0"/>
+    <origin xyz="0.02 0.61 -0.32" rpy="0.0 -0.0 0.0" />
+    <parent link="TFRAME" />
+    <child link="TRACK_L" />
+  </joint>
+  <link name="TRACK_R"/>
+  <joint name="TRACK_R" type="continuous">
+    <axis xyz="0 -1 0"/>
+    <origin xyz="0.02 -0.61 -0.32" rpy="0.0 -0.0 0.0" />
+    <parent link="TFRAME" />
+    <child link="TRACK_R" />
+  </joint>
+  <!-- Transmission -->
+  <xacro:joint_velocity_trans_v0 name="TRACK_L"/>
+  <xacro:joint_velocity_trans_v0 name="TRACK_R"/>
 </robot>
