Commit message: Update to rtr tip link

File: rtr_double_arm_v7_description/urdf/TOHOKU_ARM.urdf.xacro (robot description, xacro)
@@ -146,11 +146,13 @@
       <material name="tohku_tip_color"/>
       <geometry>
-        <mesh filename="package://rtr_double_arm_v7_description/meshes/tohku_hand_tip.stl"/>
-      </geometry>
-    </visual>
-    <collision>
-      <origin rpy="${-M_PI/2} ${-M_PI/2} 0"/>
-      <geometry>
-        <mesh filename="package://rtr_double_arm_v7_description/meshes/tohku_hand_tip.stl"/>
+        <!-- <mesh filename="package://rtr_double_arm_v7_description/meshes/tohku_hand_tip.stl"/> -->
+        <mesh filename="package://rtr_double_arm_v7_description/meshes/rtr_tip_01.stl"/>
+      </geometry>
+    </visual>
+    <collision>
+      <origin rpy="${-M_PI/2} ${-M_PI/2} 0"/>
+      <geometry>
+        <!-- <mesh filename="package://rtr_double_arm_v7_description/meshes/tohku_hand_tip.stl"/> -->
+        <mesh filename="package://rtr_double_arm_v7_description/meshes/rtr_tip_01.stl"/>
       </geometry>
     </collision>
@@ -166,11 +168,13 @@
       <material name="tohku_tip_color"/>
       <geometry>
-        <mesh filename="package://rtr_double_arm_v7_description/meshes/tohku_hand_tip.stl"/>
-      </geometry>
-    </visual>
-    <collision>
-      <origin rpy="${-M_PI/2} ${-M_PI/2} 0"/>
-      <geometry>
-        <mesh filename="package://rtr_double_arm_v7_description/meshes/tohku_hand_tip.stl"/>
+        <!-- <mesh filename="package://rtr_double_arm_v7_description/meshes/tohku_hand_tip.stl"/> -->
+        <mesh filename="package://rtr_double_arm_v7_description/meshes/rtr_tip_01.stl"/>
+      </geometry>
+    </visual>
+    <collision>
+      <origin rpy="${-M_PI/2} ${-M_PI/2} 0"/>
+      <geometry>
+        <!-- <mesh filename="package://rtr_double_arm_v7_description/meshes/tohku_hand_tip.stl"/> -->
+        <mesh filename="package://rtr_double_arm_v7_description/meshes/rtr_tip_01.stl"/>
       </geometry>
     </collision>

Commit message: Update to add end effector link

File: rtr_double_arm_v7_description/urdf/TOHOKU_ARM.urdf.xacro (robot description, xacro)
@@ -185,4 +185,5 @@
     </inertial>
   </link>
+  <link name="TOHKU_EEF"/>
   <!-- Joint -->
   <joint name="MFRAME" type="revolute">
@@ -242,3 +243,8 @@
     <limit lower="-0.349065850399" upper="0.0" effort="10000.0" velocity="573.0" />
   </joint>
+  <joint name="TOHKU_EEF" type="fixed">
+    <origin xyz="0 0 -0.735" rpy="0.0 -0.0 0.0" />
+    <parent link="TOHKU_ROLL" />
+    <child link="TOHKU_EEF" />
+  </joint>
 </robot>
