Commit message: Update base frame shape

File: rtr_double_arm_v7_description/urdf/MANI_ARM.urdf.xacro (robot description, xacro)
@@ -48,5 +48,5 @@
       <material name="uframe_color"/>
       <geometry>
-        <mesh filename="package://rtr_double_arm_v7_description/meshes/frame_marge.stl"/>
+        <mesh filename="package://rtr_double_arm_v7_description/meshes/frame_marge.dae"/>
       </geometry>
     </visual>
@@ -54,5 +54,5 @@
       <origin rpy="${M_PI/2} 0 0"/>
       <geometry>
-        <mesh filename="package://rtr_double_arm_v7_description/meshes/frame_marge.stl"/>
+        <mesh filename="package://rtr_double_arm_v7_description/meshes/frame_marge.dae"/>
       </geometry>
     </collision>
