Commit message: Update to add Camera frames

File: rtr_double_arm_v7_description/urdf/SENSOR.urdf.xacro (robot description, xacro)
@@ -7,4 +7,100 @@
     <child link="Velodyne"/>
   </joint>
+  <link name="Camera00"/>
+  <joint name="Camera00" type="fixed">
+    <origin xyz="0.475 0 1.175" rpy="${M_PI/2} ${-80*M_PI/180} 0"/>
+    <parent link="TFRAME"/>
+    <child link="Camera00"/>
+  </joint>
+  <link name="Camera01"/>
+  <joint name="Camera01" type="fixed">
+    <origin xyz="0.55 0 1.175" rpy="${M_PI/2} ${-45*M_PI/180} 0"/>
+    <parent link="TFRAME"/>
+    <child link="Camera01"/>
+  </joint>
+  <link name="Camera02"/>
+  <joint name="Camera02" type="fixed">
+    <origin xyz="0.3358 0.3358 1.175" rpy="${M_PI/2} ${-80*M_PI/180} ${45*M_PI/180}"/>
+    <parent link="TFRAME"/>
+    <child link="Camera02"/>
+  </joint>
+  <link name="Camera03"/>
+  <joint name="Camera03" type="fixed">
+    <origin xyz="0.3889 0.3889 1.175" rpy="${M_PI/2} ${-45*M_PI/180} ${45*M_PI/180}"/>
+    <parent link="TFRAME"/>
+    <child link="Camera03"/>
+  </joint>
+  <link name="Camera04"/>
+  <joint name="Camera04" type="fixed">
+    <origin xyz="0 0.475 1.175" rpy="${M_PI/2} ${-80*M_PI/180} ${90*M_PI/180}"/>
+    <parent link="TFRAME"/>
+    <child link="Camera04"/>
+  </joint>
+  <link name="Camera05"/>
+  <joint name="Camera05" type="fixed">
+    <origin xyz="0 0.55 1.175" rpy="${M_PI/2} ${-45*M_PI/180} ${90*M_PI/180}"/>
+    <parent link="TFRAME"/>
+    <child link="Camera05"/>
+  </joint>
+  <link name="Camera06"/>
+  <joint name="Camera06" type="fixed">
+    <origin xyz="-0.3358 0.3358 1.175" rpy="${M_PI/2} ${-80*M_PI/180} ${135*M_PI/180}"/>
+    <parent link="TFRAME"/>
+    <child link="Camera06"/>
+  </joint>
+  <link name="Camera07"/>
+  <joint name="Camera07" type="fixed">
+    <origin xyz="-0.3889 0.3889 1.175" rpy="${M_PI/2} ${-45*M_PI/180} ${135*M_PI/180}"/>
+    <parent link="TFRAME"/>
+    <child link="Camera07"/>
+  </joint>
+  <link name="Camera08"/>
+  <joint name="Camera08" type="fixed">
+    <origin xyz="-0.475 0 1.175" rpy="${M_PI/2} ${-80*M_PI/180} ${180*M_PI/180}"/>
+    <parent link="TFRAME"/>
+    <child link="Camera08"/>
+  </joint>
+  <link name="Camera09"/>
+  <joint name="Camera09" type="fixed">
+    <origin xyz="-0.55 0 1.175" rpy="${M_PI/2} ${-45*M_PI/180} ${180*M_PI/180}"/>
+    <parent link="TFRAME"/>
+    <child link="Camera09"/>
+  </joint>
+  <link name="Camera10"/>
+  <joint name="Camera10" type="fixed">
+    <origin xyz="-0.3358 -0.3358 1.175" rpy="${M_PI/2} ${-80*M_PI/180} ${225*M_PI/180}"/>
+    <parent link="TFRAME"/>
+    <child link="Camera10"/>
+  </joint>
+  <link name="Camera11"/>
+  <joint name="Camera11" type="fixed">
+    <origin xyz="-0.3889 -0.3889 1.175" rpy="${M_PI/2} ${-45*M_PI/180} ${225*M_PI/180}"/>
+    <parent link="TFRAME"/>
+    <child link="Camera11"/>
+  </joint>
+  <link name="Camera12"/>
+  <joint name="Camera12" type="fixed">
+    <origin xyz="0 -0.475 1.175" rpy="${M_PI/2} ${-80*M_PI/180} ${270*M_PI/180}"/>
+    <parent link="TFRAME"/>
+    <child link="Camera12"/>
+  </joint>
+  <link name="Camera13"/>
+  <joint name="Camera13" type="fixed">
+    <origin xyz="0 -0.55 1.175" rpy="${M_PI/2} ${-45*M_PI/180} ${270*M_PI/180}"/>
+    <parent link="TFRAME"/>
+    <child link="Camera13"/>
+  </joint>
+  <link name="Camera14"/>
+  <joint name="Camera14" type="fixed">
+    <origin xyz="0.3358 -0.3358 1.175" rpy="${M_PI/2} ${-80*M_PI/180} ${315*M_PI/180}"/>
+    <parent link="TFRAME"/>
+    <child link="Camera14"/>
+  </joint>
+  <link name="Camera15"/>
+  <joint name="Camera15" type="fixed">
+    <origin xyz="0.3889 -0.3889 1.175" rpy="${M_PI/2} ${-45*M_PI/180} ${315*M_PI/180}"/>
+    <parent link="TFRAME"/>
+    <child link="Camera15"/>
+  </joint>
 <!-- <link name="SWING_TORQUE"> -->
 <!--   </link> -->

Commit message: Updating to add depth sensor

File: rtr_double_arm_v7_description/urdf/SENSOR.urdf.xacro (robot description, xacro)
@@ -103,4 +103,10 @@
     <child link="Camera15"/>
   </joint>
+  <link name="TohokuDepthCamera00"/>
+  <joint name="TohokuDepthCamera00" type="fixed">
+    <origin xyz="0 0 0" rpy="${90*M_PI/180} ${-90*M_PI/180} 0"/>
+    <parent link="TOHKU_ROLL"/>
+    <child link="TohokuDepthCamera00"/>
+  </joint>
 <!-- <link name="SWING_TORQUE"> -->
 <!--   </link> -->

Commit message: Update Tohoku & Mani grippter depth camera pose

File: rtr_double_arm_v7_description/urdf/SENSOR.urdf.xacro (robot description, xacro)
@@ -105,128 +105,37 @@
   <link name="TohokuDepthCamera00"/>
   <joint name="TohokuDepthCamera00" type="fixed">
-    <origin xyz="0 0 0" rpy="${90*M_PI/180} ${-90*M_PI/180} 0"/>
+    <origin xyz="0 0.2 -0.2" rpy="${-90*M_PI/180} 0 0"/>
     <parent link="TOHKU_ROLL"/>
     <child link="TohokuDepthCamera00"/>
   </joint>
-<!-- <link name="SWING_TORQUE"> -->
-<!--   </link> -->
-<!--   <joint name="SWING_TORQUE_JOINT" type="fixed"> -->
-<!--     <origin xyz="0.0 0.0 0.0" rpy="0.0 -0.0 0.0" /> -->
-<!--     <parent link="BLOCK" /> -->
-<!--     <child link="SWING_TORQUE" /> -->
-<!--   </joint> -->
-<!--   <sensor name="SWING_TORQUE_SENSOR" update_rate="20"> -->
-<!--     <origin xyz="0.0 0.0 0.0" rpy="0.0 -0.0 0.0" /> -->
-<!--     <parent link="BLOCK" /> -->
-<!--   </sensor> -->
-<!--   <link name="BOOM_TORQUE"> -->
-<!--   </link> -->
-<!--   <joint name="BOOM_TORQUE_JOINT" type="fixed"> -->
-<!--     <origin xyz="0.0 0.0 0.0" rpy="1.57079632679 7.14632589097e-16 3.14159265359" /> -->
-<!--     <parent link="BOOM" /> -->
-<!--     <child link="BOOM_TORQUE" /> -->
-<!--   </joint> -->
-<!--   <sensor name="BOOM_TORQUE_SENSOR" update_rate="20"> -->
-<!--     <origin xyz="0.0 0.0 0.0" rpy="1.57079632679 7.14632589097e-16 3.14159265359" /> -->
-<!--     <parent link="BOOM" /> -->
-<!--   </sensor> -->
-<!--   <link name="ARM_TORQUE"> -->
-<!--   </link> -->
-<!--   <joint name="ARM_TORQUE_JOINT" type="fixed"> -->
-<!--     <origin xyz="0.0 0.0 0.0" rpy="1.57079632679 7.14632589097e-16 3.14159265359" /> -->
-<!--     <parent link="ARM" /> -->
-<!--     <child link="ARM_TORQUE" /> -->
-<!--   </joint> -->
-<!--   <sensor name="ARM_TORQUE_SENSOR" update_rate="20"> -->
-<!--     <origin xyz="0.0 0.0 0.0" rpy="1.57079632679 7.14632589097e-16 3.14159265359" /> -->
-<!--     <parent link="ARM" /> -->
-<!--   </sensor> -->
-<!--   <link name="HAND_P_TORQUE"> -->
-<!--   </link> -->
-<!--   <joint name="HAND_P_TORQUE_JOINT" type="fixed"> -->
-<!--     <origin xyz="0.0 0.0 0.0" rpy="1.57079632679 7.14632589097e-16 3.14159265359" /> -->
-<!--     <parent link="TOHKU_PITCH" /> -->
-<!--     <child link="HAND_P_TORQUE" /> -->
-<!--   </joint> -->
-<!--   <sensor name="HAND_P_TORQUE_SENSOR" update_rate="20"> -->
-<!--     <origin xyz="0.0 0.0 0.0" rpy="1.57079632679 7.14632589097e-16 3.14159265359" /> -->
-<!--     <parent link="TOHKU_PITCH" /> -->
-<!--   </sensor> -->
-<!--   <link name="MNP_SWING_TORQUE"> -->
-<!--   </link> -->
-<!--   <joint name="MNP_SWING_TORQUE_JOINT" type="fixed"> -->
-<!--     <origin xyz="0.0 0.0 0.0" rpy="1.57079632679 -0.0 1.57079632679" /> -->
-<!--     <parent link="MNP_SWING" /> -->
-<!--     <child link="MNP_SWING_TORQUE" /> -->
-<!--   </joint> -->
-<!--   <sensor name="MNP_SWING_TORQUE_SENSOR" update_rate="20"> -->
-<!--     <origin xyz="0.0 0.0 0.0" rpy="1.57079632679 -0.0 1.57079632679" /> -->
-<!--     <parent link="MNP_SWING" /> -->
-<!--   </sensor> -->
-<!--   <link name="MNP_BOOM_TORQUE"> -->
-<!--   </link> -->
-<!--   <joint name="MNP_BOOM_TORQUE_JOINT" type="fixed"> -->
-<!--     <origin xyz="0.0 0.0 0.0" rpy="7.8859849469e-16 9.95799250103e-17 -1.57079632679" /> -->
-<!--     <parent link="MANIBOOM" /> -->
-<!--     <child link="MNP_BOOM_TORQUE" /> -->
-<!--   </joint> -->
-<!--   <sensor name="MNP_BOOM_TORQUE_SENSOR" update_rate="20"> -->
-<!--     <origin xyz="0.0 0.0 0.0" rpy="7.8859849469e-16 9.95799250103e-17 -1.57079632679" /> -->
-<!--     <parent link="MANIBOOM" /> -->
-<!--   </sensor> -->
-<!--   <link name="MNP_ARM_TORQUE"> -->
-<!--   </link> -->
-<!--   <joint name="MNP_ARM_TORQUE_JOINT" type="fixed"> -->
-<!--     <origin xyz="0.0 0.0 0.0" rpy="7.8859849469e-16 9.95799250103e-17 -1.57079632679" /> -->
-<!--     <parent link="MANIARM" /> -->
-<!--     <child link="MNP_ARM_TORQUE" /> -->
-<!--   </joint> -->
-<!--   <sensor name="MNP_ARM_TORQUE_SENSOR" update_rate="20"> -->
-<!--     <origin xyz="0.0 0.0 0.0" rpy="7.8859849469e-16 9.95799250103e-17 -1.57079632679" /> -->
-<!--     <parent link="MANIARM" /> -->
-<!--   </sensor> -->
-<!--   <link name="MNP_ELBOW_TORQUE"> -->
-<!--   </link> -->
-<!--   <joint name="MNP_ELBOW_TORQUE_JOINT" type="fixed"> -->
-<!--     <origin xyz="0.0 0.0 0.0" rpy="7.8859849469e-16 9.95799250103e-17 -1.57079632679" /> -->
-<!--     <parent link="MANIELBOW" /> -->
-<!--     <child link="MNP_ELBOW_TORQUE" /> -->
-<!--   </joint> -->
-<!--   <sensor name="MNP_ELBOW_TORQUE_SENSOR" update_rate="20"> -->
-<!--     <origin xyz="0.0 0.0 0.0" rpy="7.8859849469e-16 9.95799250103e-17 -1.57079632679" /> -->
-<!--     <parent link="MANIELBOW" /> -->
-<!--   </sensor> -->
-<!--   <link name="MNP_YAW_TORQUE"> -->
-<!--   </link> -->
-<!--   <joint name="MNP_YAW_TORQUE_JOINT" type="fixed"> -->
-<!--     <origin xyz="0.0 0.0 0.0" rpy="3.14159265359 -1.57079632679 0.0" /> -->
-<!--     <parent link="YAWJOINT" /> -->
-<!--     <child link="MNP_YAW_TORQUE" /> -->
-<!--   </joint> -->
-<!--   <sensor name="MNP_YAW_TORQUE_SENSOR" update_rate="20"> -->
-<!--     <origin xyz="0.0 0.0 0.0" rpy="3.14159265359 -1.57079632679 0.0" /> -->
-<!--     <parent link="YAWJOINT" /> -->
-<!--   </sensor> -->
-<!--   <link name="MNP_ROLL_TORQUE"> -->
-<!--   </link> -->
-<!--   <joint name="MNP_ROLL_TORQUE_JOINT" type="fixed"> -->
-<!--     <origin xyz="0.0 0.0 0.0" rpy="1.57079632679 -2.88998133609e-16 -3.00440511061e-16" /> -->
-<!--     <parent link="HANDBASE" /> -->
-<!--     <child link="MNP_ROLL_TORQUE" /> -->
-<!--   </joint> -->
-<!--   <sensor name="MNP_ROLL_TORQUE_SENSOR" update_rate="20"> -->
-<!--     <origin xyz="0.0 0.0 0.0" rpy="1.57079632679 -2.88998133609e-16 -3.00440511061e-16" /> -->
-<!--     <parent link="HANDBASE" /> -->
-<!--   </sensor> -->
-<!--   <link name="MNP_PUSH_FORCE"> -->
-<!--   </link> -->
-<!--   <joint name="MNP_PUSH_FORCE_JOINT" type="fixed"> -->
-<!--     <origin xyz="0.0 0.0 0.0" rpy="0.0 -0.0 0.0" /> -->
-<!--     <parent link="PUSHROD" /> -->
-<!--     <child link="MNP_PUSH_FORCE" /> -->
-<!--   </joint> -->
-<!--   <sensor name="MNP_PUSH_FORCE_SENSOR" update_rate="20"> -->
-<!--     <origin xyz="0.0 0.0 0.0" rpy="0.0 -0.0 0.0" /> -->
-<!--     <parent link="PUSHROD" /> -->
-<!--   </sensor> -->
+  <!-- <link name="TohokuDepthCamera01"/> -->
+  <!-- <joint name="TohokuDepthCamera01" type="fixed"> -->
+  <!--   <origin xyz="0.2 0 -0.2" rpy="${-90*M_PI/180} 0 ${-90*M_PI/180}"/> -->
+  <!--   <parent link="TOHKU_ROLL"/> -->
+  <!--   <child link="TohokuDepthCamera01"/> -->
+  <!-- </joint> -->
+  <link name="TohokuDepthCamera02"/>
+  <joint name="TohokuDepthCamera02" type="fixed">
+    <origin xyz="0 -0.2 -0.2" rpy="0 ${M_PI} 0"/>
+    <parent link="TOHKU_ROLL"/>
+    <child link="TohokuDepthCamera02"/>
+  </joint>
+  <!-- <link name="TohokuDepthCamera03"/> -->
+  <!-- <joint name="TohokuDepthCamera03" type="fixed"> -->
+  <!--   <origin xyz="0 -0.2 -0.2" rpy="0 ${M_PI} 0"/>  -->
+  <!--   <parent link="TOHKU_ROLL"/> -->
+  <!--   <child link="TohokuDepthCamera03"/> -->
+  <!-- </joint> -->
+  <link name="ManiDepthCamera00"/>
+  <joint name="ManiDepthCamera00" type="fixed">
+    <origin xyz="0 0.3 -0.1" rpy="${180*M_PI/180} 0 0"/>
+    <parent link="HANDBASE"/>
+    <child link="ManiDepthCamera00"/>
+  </joint>
+  <link name="ManiDepthCamera02"/>
+  <joint name="ManiDepthCamera02" type="fixed">
+    <origin xyz="0 -0.3 -0.1" rpy="0 ${M_PI} 0"/>
+    <parent link="HANDBASE"/>
+    <child link="ManiDepthCamera02"/>
+  </joint>
 </robot>

Commit message: Update camera positions/orientations

File: rtr_double_arm_v7_description/urdf/SENSOR.urdf.xacro (robot description, xacro)
@@ -105,37 +105,25 @@
   <link name="TohokuDepthCamera00"/>
   <joint name="TohokuDepthCamera00" type="fixed">
-    <origin xyz="0 0.2 -0.2" rpy="${-90*M_PI/180} 0 0"/>
+    <origin xyz="0 0.2 -0.2" rpy="0 ${M_PI} ${M_PI}"/>
     <parent link="TOHKU_ROLL"/>
     <child link="TohokuDepthCamera00"/>
   </joint>
-  <!-- <link name="TohokuDepthCamera01"/> -->
-  <!-- <joint name="TohokuDepthCamera01" type="fixed"> -->
-  <!--   <origin xyz="0.2 0 -0.2" rpy="${-90*M_PI/180} 0 ${-90*M_PI/180}"/> -->
-  <!--   <parent link="TOHKU_ROLL"/> -->
-  <!--   <child link="TohokuDepthCamera01"/> -->
-  <!-- </joint> -->
-  <link name="TohokuDepthCamera02"/>
-  <joint name="TohokuDepthCamera02" type="fixed">
+  <link name="TohokuDepthCamera01"/>
+  <joint name="TohokuDepthCamera01" type="fixed">
     <origin xyz="0 -0.2 -0.2" rpy="0 ${M_PI} 0"/>
     <parent link="TOHKU_ROLL"/>
-    <child link="TohokuDepthCamera02"/>
+    <child link="TohokuDepthCamera01"/>
   </joint>
-  <!-- <link name="TohokuDepthCamera03"/> -->
-  <!-- <joint name="TohokuDepthCamera03" type="fixed"> -->
-  <!--   <origin xyz="0 -0.2 -0.2" rpy="0 ${M_PI} 0"/>  -->
-  <!--   <parent link="TOHKU_ROLL"/> -->
-  <!--   <child link="TohokuDepthCamera03"/> -->
-  <!-- </joint> -->
   <link name="ManiDepthCamera00"/>
   <joint name="ManiDepthCamera00" type="fixed">
-    <origin xyz="0 0.3 -0.1" rpy="${180*M_PI/180} 0 0"/>
+    <origin xyz="0 0.1 -0.3" rpy="0 ${M_PI} ${M_PI}"/>
     <parent link="HANDBASE"/>
     <child link="ManiDepthCamera00"/>
   </joint>
-  <link name="ManiDepthCamera02"/>
-  <joint name="ManiDepthCamera02" type="fixed">
-    <origin xyz="0 -0.3 -0.1" rpy="0 ${M_PI} 0"/>
+  <link name="ManiDepthCamera01"/>
+  <joint name="ManiDepthCamera01" type="fixed">
+    <origin xyz="0 -0.1 -0.3" rpy="0 ${M_PI} 0"/>
     <parent link="HANDBASE"/>
-    <child link="ManiDepthCamera02"/>
+    <child link="ManiDepthCamera01"/>
   </joint>
 </robot>
