Commit message: Add range sensor to quadcopter

File: rtr_quadcopter_description/xacro/rtr_quadcopter_wrs.urdf.xacro (robot description, xacro)
@@ -56,4 +56,34 @@
     </visual>
   </link>
+  <joint name="UpperRangeSensorJoint" type="fixed">
+    <parent link="BODY"/>
+    <child link="UpperRangeSensor"/>
+    <origin xyz="0.00 0 0.05" rpy="0 0 0"/>
+  </joint>
+  <link name="UpperRangeSensor">
+    <visual>
+      <geometry>
+        <cylinder radius="0.003" length="0.01"/>
+      </geometry>
+      <material name="red">
+        <color rgba="1.0 0.0 0.0 1.0"/>
+      </material>
+    </visual>
+  </link>
+  <joint name="LowerRangeSensorJoint" type="fixed">
+    <parent link="BODY"/>
+    <child link="LowerRangeSensor"/>
+    <origin xyz="0.00 0 -0.05" rpy="0 0 0"/>
+  </joint>
+  <link name="LowerRangeSensor">
+    <visual>
+      <geometry>
+        <cylinder radius="0.003" length="0.01"/>
+      </geometry>
+      <material name="red">
+        <color rgba="1.0 0.0 0.0 1.0"/>
+      </material>
+    </visual>
+  </link>
   <!-- Legs -->
   <xacro:macro name="leg" params="name translation">

Commit message: Add fixed xacro

File: rtr_quadcopter_description/xacro/rtr_quadcopter_wrs.urdf.xacro (robot description, xacro)
@@ -1,3 +1,4 @@
-<robot name="quadcopter_wrs" xmlns:xacro="http://ros.org/wiki/xacro">
+<robot name="quadcopter_wrs"
+  xmlns:xacro="http://ros.org/wiki/xacro">
   <xacro:property name="side" value="0.5"/>
   <link name="BODY">
@@ -12,12 +13,19 @@
     </visual>
   </link>
-  <joint name="CAMERA_T" type="revolute">
-    <parent link="BODY"/>
-    <child link="CAMERA_T"/>
+  <joint name="CAMERA_2" type="revolute">
+    <parent link="BODY"/>
+    <child link="CAMERA_2"/>
     <origin xyz="0 0 -0.05"/>
     <limit lower="${-pi}" upper="0" velocity="${pi/2}" effort="1"/>
     <axis xyz="0 -1 0"/>
   </joint>
-  <link name="CAMERA_T">
+  <joint name="CAMERA_3" type="revolute">
+    <parent link="BODY"/>
+    <child link="CAMERA_3"/>
+    <origin xyz="0 0 0.10"/>
+    <limit lower="${-pi}" upper="0" velocity="${pi/2}" effort="1"/>
+    <axis xyz="0 -1 0"/>
+  </joint>
+  <link name="CAMERA_2">
     <visual>
       <origin rpy="0 0 0" xyz="0 0 0"/>
@@ -29,5 +37,5 @@
   </link>
   <joint name="CameraJoint" type="fixed">
-    <parent link="CAMERA_T"/>
+    <parent link="CAMERA_2"/>
     <child link="Camera"/>
     <origin xyz="0.03 0 0" rpy="${-pi/2} 0 ${-pi/2}"/>
@@ -44,5 +52,5 @@
   </link>
   <joint name="Camera2Joint" type="fixed">
-    <parent link="CAMERA_T"/>
+    <parent link="CAMERA_2"/>
     <child link="Camera2"/>
     <origin xyz="0.02 0 -0.02" rpy="${-pi/2} 0 ${-pi/2}"/>
@@ -71,17 +79,31 @@
     </visual>
   </link>
-  <joint name="LowerRangeSensorJoint" type="fixed">
-    <parent link="BODY"/>
-    <child link="LowerRangeSensor"/>
-    <origin xyz="0.00 0 -0.05" rpy="0 0 0"/>
-  </joint>
-  <link name="LowerRangeSensor">
-    <visual>
-      <geometry>
-        <cylinder radius="0.003" length="0.01"/>
-      </geometry>
-      <material name="red">
-        <color rgba="1.0 0.0 0.0 1.0"/>
-      </material>
+  <!-- <joint name="CAMERA_3" type="revolute">
+    <parent link="BODY"/>
+    <child link="Camera3"/>
+    <origin xyz="0 0 0.10"/>
+    <limit lower="${-pi}" upper="0" velocity="${pi/2}" effort="1"/>
+    <axis xyz="0 -1 0"/>
+  </joint> -->
+  <link name="CAMERA_3">
+    <visual>
+      <origin rpy="0 0 0" xyz="0 0 0"/>
+      <geometry>
+        <sphere radius="0.03"/>
+      </geometry>
+      <material name="blue"/>
+    </visual>
+  </link>
+  <joint name="Camera3Joint" type="fixed">
+    <parent link="CAMERA_3"/>
+    <child link="Camera3"/>
+    <origin xyz="0.02 0 0.02" rpy="${-pi/2} 0 ${-pi/2}"/>
+  </joint>
+  <link name="Camera3">
+    <visual>
+      <geometry>
+        <cylinder radius="0.003" length="0.01"/>
+      </geometry>
+      <material name="red"/>
     </visual>
   </link>
